Commit message: Followed panda_moveit_config for moveit integration

File: src/rbkairos_common/rbkairos_description/robots/versions/rbkairos_panda_hand.urdf.xacro (robot description, xacro)
@@ -30,5 +30,5 @@
   <xacro:property name="arm_orientation_r" value="0"/>
   <xacro:property name="arm_orientation_p" value="0"/>
-  <xacro:property name="arm_orientation_y" value="${4*pi/4}"/>
+  <xacro:property name="arm_orientation_y" value="0"/>
   <xacro:macro name="rbkairos_panda_hand" params="prefix publish_bf hq load_kinematics_file gpu:=false">
     <!-- *************** -->
@@ -70,5 +70,4 @@
     <xacro:gazebo-joint joint="${arm_id}_joint6" transmission="hardware_interface/PositionJointInterface" />
     <xacro:gazebo-joint joint="${arm_id}_joint7" transmission="hardware_interface/PositionJointInterface" />
-    <!--
     <xacro:gazebo-joint joint="${arm_id}_joint1" transmission="hardware_interface/VelocityJointInterface" />
     <xacro:gazebo-joint joint="${arm_id}_joint2" transmission="hardware_interface/VelocityJointInterface" />
@@ -78,5 +77,4 @@
     <xacro:gazebo-joint joint="${arm_id}_joint6" transmission="hardware_interface/VelocityJointInterface" />
     <xacro:gazebo-joint joint="${arm_id}_joint7" transmission="hardware_interface/VelocityJointInterface" />
-    -->
     <xacro:gazebo-joint joint="${arm_id}_joint1" transmission="hardware_interface/EffortJointInterface" />
     <xacro:gazebo-joint joint="${arm_id}_joint2" transmission="hardware_interface/EffortJointInterface" />
